Commit message: ruedas giradas nitidamente

File: urdf/robot.urdf (robot description, URDF)
Before this commit: robot robot, 11 links, 10 joints
Joints:
- joint back_left_wheel_joint: origin xyz=1.724564 -0.893577 -1.584369 rpy=1.570796 1.570796 0 -> xyz=-1.724564 -0.893577 -1.584369 rpy=1.570796 1.570796 3.141593
- joint back_right_wheel_joint: origin xyz=1.724564 0.893577 -1.584369 rpy=1.570796 1.570796 0 -> xyz=-1.724564 0.893577 -1.584369 rpy=1.570796 1.570796 3.141593
- joint front_left_wheel_joint: origin xyz=-0.859709 -0.893577 -1.584369 rpy=1.570796 1.570796 0 -> xyz=0.859709 -0.893577 -1.584369 rpy=1.570796 1.570796 3.141593
- joint front_right_wheel_joint: origin xyz=-0.859709 0.893577 -1.584369 rpy=1.570796 1.570796 0 -> xyz=0.859709 0.893577 -1.584369 rpy=1.570796 1.570796 3.141593

Commit message: robot con giro de 180º!!!!!!! falta sensores

File: urdf/robot.urdf (robot description, URDF)
Before this commit: robot robot, 11 links, 10 joints
Joints:
- joint arm1_joint: origin xyz=-0.053901 0 0.102658 rpy=1.570796 1.570796 0 -> xyz=0.053901 0 0.102658 rpy=-1.570796 1.570796 0
- joint arm2_joint: origin xyz=-1.544378 -0.000489 -0.000415 rpy=0 0 0 -> xyz=-1.544378 -0.000489 0.000415 rpy=0 0 0
- joint arm_base_joint: origin xyz=-1.24578 0 0.535008 rpy=0 0 0 -> xyz=1.24578 0 0.535008 rpy=0 0 0

Commit message: rep103

File: urdf/robot.urdf (robot description, URDF)
Before this commit: robot robot, 11 links, 10 joints
Joints:
- joint back_left_wheel_joint: origin xyz=-1.724564 -0.893577 -1.584369 rpy=1.570796 1.570796 3.141593 -> xyz=-1.724564 -0.893577 -1.584369 rpy=1.570796 0 0
- joint back_right_wheel_joint: origin xyz=-1.724564 0.893577 -1.584369 rpy=1.570796 1.570796 3.141593 -> xyz=-1.724564 0.893577 -1.584369 rpy=1.570796 3.141593 3.141593
- joint front_left_wheel_joint: origin xyz=0.859709 -0.893577 -1.584369 rpy=1.570796 1.570796 3.141593 -> xyz=0.859709 -0.893577 -1.584369 rpy=1.570796 0 0
- joint front_right_wheel_joint: origin xyz=0.859709 0.893577 -1.584369 rpy=1.570796 1.570796 3.141593 -> xyz=0.859709 0.893577 -1.584369 rpy=1.570796 3.141593 3.141593

Commit message: basefootprint boff esto es un no parar

File: urdf/robot.urdf (robot description, URDF)
Before this commit: robot robot, 11 links, 10 joints
Links:
- added link base_footprint
Joints:
- added joint base_footprint_joint: type fixed, parent base_footprint, child root, origin xyz=0 0 1.9 rpy=0 0 0

Commit message: quité el bracito

File: urdf/robot.urdf (robot description, URDF)
Before this commit: robot robot, 12 links, 11 joints
Links:
- removed link arm1_link
- removed link arm2_link
- removed link arm3_link
- removed link arm_base_link
- removed link left_gripper_link
- removed link right_gripper_link
Joints:
- removed joint arm1_joint
- removed joint arm2_joint
- removed joint arm3_joint
- removed joint arm_base_joint
- removed joint left_gripper_joint
- removed joint right_gripper_joint
